File: pcb_phone_controller/pcb_phone_controller.kicad_sch (KiCad schematic)
At the start: 38 parts, among them SW17 SS-12D00-G 4 E, X1 KAILH-MINI-SILENT-SWITCH, Y1 KAILH-MINI-SILENT-SWITCH

Commit message: PCB cleanup (libs and traces)
Parts:
- removed TriggerL1, TriggerR1: SS49E, CC-Library:SEN3_SS49E_HNW, symbol SS49E:SS49E
- added TriggerL1, TriggerR1: SS49E, Lib_controller:ss49e, symbol Lib_controller:SS49E
- +-1: footprint CC-Library:Battery_connection -> Lib_controller:Battery_connection; symbol CC-Library:Battery_connection -> Lib_controller:Battery_connection
- A1, B1, DOWN1, Home1, LEFT1, RIGHT1, Select1, Start1, UP1, X1, Y1: footprint CC-Library:KAILH-MINI-SILENT-SWITCH -> Lib_controller:KAILH-MINI-SILENT-SWITCH; symbol CC-Library:KAILH-MINI-SILENT-SWITCH -> Lib_controller:KAILH-MINI-SILENT-SWITCH
- BumperL1, BumperR1, ClickStickL1, ClickStickR1: footprint CC-Library:PinHeader_1x03_P2.54mm_Vertical -> Lib_controller:PinHeader_1x03_P2.54mm_Vertical
- SW17: footprint CC-Library:1P2T_SS-12D00_CNK -> Lib_controller:1P2T_SS-12D00_CNK; symbol CC-Library:SS-12D00-G_4_E -> Lib_controller:SS-12D00-G_4_E
- StickL1, StickR1: symbol CC-Library:SM-3ds-stick -> Lib_controller:3DS_stick
- U1: footprint CC-Library:Seeed Studio XIAO ESP32S3 Plus -> Lib_controller:Seeed Studio XIAO ESP32S3 Plus; symbol CC-Library:Seeed_Studio_XIAO_ESP32S3_Plus -> Lib_controller:Seeed_Studio_XIAO_ESP32S3_Plus
Connections:
- net +3.3V: now also TriggerL1.1 (VDD), TriggerR1.1 (VDD)
- net GND: now also TriggerL1.2 (GND), TriggerR1.2 (GND)
- net at U1.6 (GPIO): now also TriggerL1.3 (OUT)
- net at U1.9 (GPIO): now also TriggerR1.3 (OUT)
